Commit message: modified basic comments staged misssed filed
Former-commit-id: 9ce943bddb27da5e9b4805602d090609bb5a19f9
Former-commit-id: 778d6f160603d36771a4817da918222908d9150c

File: dimos/hardware/piper_description.urdf (robot description, URDF)
Before this commit: robot piper, 10 links, 9 joints
Links:
- removed link link7
- removed link link8
- link base_link: mass 1.02 -> 1; geometry collision box size=0.08 0.08 0.04; visual box size=0.08 0.08 0.04
- link gripper_base: mass 0.45 -> None; geometry collision box size=0.03 0.03 0.04; visual box size=0.03 0.03 0.04
- link link1: mass 0.71 -> None; geometry collision box size=0.05 0.05 0.1; visual box size=0.05 0.05 0.1
- link link2: mass 1.17 -> None; geometry collision box size=0.05 0.05 0.16; visual box size=0.05 0.05 0.16
- link link3: mass 0.5 -> None; geometry collision box size=0.05 0.05 0.16; visual box size=0.05 0.05 0.16
- link link4: mass 0.38 -> None; geometry collision box size=0.045 0.045 0.12; visual box size=0.045 0.045 0.12
- link link5: mass 0.383 -> None; geometry collision box size=0.04 0.04 0.08; visual box size=0.04 0.04 0.08
- link link6: mass 0.00699089613564366 -> None; geometry collision box size=0.035 0.035 0.06; visual box size=0.035 0.035 0.06
Joints:
- removed joint joint6_to_gripper_base
- removed joint joint7
- removed joint joint8
- added joint ee_fixed: type fixed, parent link6, child gripper_base, origin xyz=0 0 0.06
- joint joint1: limit lower=-2.618 upper=2.168 effort=100 velocity=5 -> lower=-3.14 upper=3.14 effort=10 velocity=2.0; origin xyz=0 0 0.123 rpy=0 0 0 -> xyz=0 0 0.02
- joint joint2: axis 0 0 1 -> 0 1 0; limit lower=0 upper=3.14 effort=100 velocity=5 -> lower=-2.1 upper=2.1 effort=10 velocity=2.0; origin xyz=0 0 0 rpy=1.5708 -0.1359 -3.1416 -> xyz=0 0 0.1
- joint joint3: axis 0 0 1 -> 0 1 0; limit lower=-2.967 upper=0 effort=100 velocity=5 -> lower=-2.8 upper=2.8 effort=10 velocity=2.0; origin xyz=0.28503 0 0 rpy=0 0 -1.7939 -> xyz=0 0 0.16
- joint joint4: axis 0 0 1 -> 1 0 0; limit lower=-1.745 upper=1.745 effort=100 velocity=5 -> lower=-3.14 upper=3.14 effort=10 velocity=2.0; origin xyz=-0.021984 -0.25075 0 rpy=1.5708 0 0 -> xyz=0 0 0.16
- joint joint5: axis 0 0 1 -> 0 1 0; limit lower=-1.22 upper=1.22 effort=100 velocity=5 -> lower=-3.14 upper=3.14 effort=10 velocity=2.0; origin xyz=0 0 0 rpy=-1.5708 0 0 -> xyz=0 0 0.12
- joint joint6: limit lower=-2.0944 upper=2.0944 effort=100 velocity=3 -> lower=-3.14 upper=3.14 effort=10 velocity=2.0; origin xyz=8.8259E-05 -0.091 0 rpy=1.5708 0 0 -> xyz=0 0 0.08
